File: pcb/kicad/Ultimate Useless Box.kicad_pcb (KiCad board)
At the start: 2 copper layers, 87.5 x 85 mm, 49 parts, among them J1 USB_C_Receptacle_USB2.0_16P, J3 Conn_01x10_Pin, Q1 S8050, U1 ESP32-S3-DevKitC, U2 DRV8833PWP, U3 TP4056-42-ESOP8, U4 MT3608

Commit message: Made changes
Parts:
- added REF**: MountingHole_2.7mm_M2.5, MountingHole:MountingHole_2.7mm_M2.5, F.Cu at (166.7, 134.5)
- added REF**: MountingHole_2.7mm_M2.5, MountingHole:MountingHole_2.7mm_M2.5, F.Cu at (89.1, 56.0)
- moved R16 1.52 mm to (161.5, 68.2), turned to -90 degrees
- moved R11 1.40 mm to (132.6, 106.1)
Routing:
- net -BATT: track 385.0 -> 373.2 mm
- net +BATT: track 151.3 -> 142.7 mm, vias 9 -> 11
- net VBUS: track 72.2 -> 77.7 mm
- net +3.3V: track 167.6 -> 163.3 mm, vias 11 -> 10
- net Net-(J1-CC1): track 5.88 -> 3.03 mm
- net Net-(J_MOT_L1-Pin_1): track 9.86 -> 11.5 mm
- net +5V: track 185.7 -> 187.1 mm
- net Net-(Q1-B): track 9.65 -> 10.6 mm
- net /VBATT_SENSE: track 149.8 -> 150.8 mm
- net Net-(J_MOT_R1-Pin_2): track 9.47 -> 8.66 mm
- net /BIN2: track 110.6 -> 111.3 mm
- added copper zone on B.Cu, net -BATT
- added copper zone on F.Cu, net -BATT
Other:
- board size 87.5 x 85 mm -> 89 x 89.7 mm
